Commit message: feat(p9-s3)!: 雷达挂高 2.2 m（S3b）+ 聚类竖向容差 1.0（S3a）—— 本地半区完成，Gazebo 全表 9/9 ×2
S3b（vehicle_params 单一来源，两环境一起动）：
- sensors.lidar.mount_z_m 1.6→2.2，SDF/URDF 重生成 --check 过；yaml 里的挂高/盲区/
  range_min 推导按 Δz=0.70 重写（最低线落地 3.43→4.72 m、近裁剪代价线 0.67→1.27 m、
  空带条件 range_min ≥ L 与 Δz 无关照旧）；动机：c3 车顶 1.571、CARLA 无近裁剪、
  1.6 时 60% 射线打自己（裸测 1.9→4%、2.2→0）
- sidecar 雷达量程改读 vehicle_params（此前写死 30 vs Gazebo 50，单一来源漏网），
  p9_lidar_probe 同源；离地阈值随挂高
- verify_ros_bridge 6/6（Δz=2.2）；文档：CLAUDE 陷阱表两行、perception.md §5/§8.2/§11、
  check_cloud_frames 注释、bringup §6 #13
S3a（共享感知）：
- euclidean_cluster 新参数 vertical_tolerance_m（1.0）：聚类前 z × tolerance/vertical
  （椭球邻域）—— 线间距顶的是竖向、1.0 m 分辨力守的是水平；25 m 处可连的进深台阶
  0.10→0.44 m、纯竖向连通极限 25.4→50.8 m；推导入 hpp/yaml/perception.md §2
- L1 +2（28 m 阶梯正面 1 簇 vs 各向同性 3 簇 —— 注入验红；并排 1.0 m 仍两簇），
  老用例反向注入补竖向同收；节点参数 cluster.vertical_tolerance_m
Gazebo 回归（新脚本 l3g_p5_round.sh = CP-P5-B 一轮一命令）：
- 1.6 基线：车 98.1%/行人 100%/近边 0.189/横向 0.327/速度 0.62/ID 4/虚警 0
- 2.2 ×3：车 98.1–99.1%/行人 100%/近边 0.14–0.18/横向 0.29–0.30/速度 0.41–0.93/
  ID 4·3·7/虚警 3·3·3（U 转鬼影：§6.5 遮挡滑行 × 重锚跳变，1.6 时落在带外；
  机理与候选修法 plan P9-4 附记，判据不放宽，待拍板）
- 2.2 + 竖向 1.0 ×3：车/行人 25–30 m 档 91.9/100/90.0 → 100/100/100%、近边
  0.14–0.17、横向 0.23–0.33、速度 0.39–0.91；ID 6/6/3、虚警 7/2/4（同上两种已知形态）
- run_all_scenarios.sh gazebo 两遍（2.2；2.2+竖向）9/9 全过
其它：L3-G test_closed_loop_obstacle 判据从 safety.margin_m（P8-S6 后 0.7）拆耦回
SPEC 0.5 —— 假车贴裕度走，0.699–0.700 骑线，一天 4 跑 3 红全是浮点噪声。
全仓 1137 tests 绿。CARLA 半区（裸测自反射、CP-P9-A ×2、CP-P9-B）待云机。

Co-Authored-By: Claude Fable 5 <noreply@anthropic.com>

File: src/ads_visualization/urdf/ego_vehicle.urdf (robot description, URDF)
Before this commit: robot ego_vehicle, 9 links, 8 joints
Joints:
- joint lidar_link_joint: origin xyz=1.3500 0.0000 1.6000 rpy=0 0 0 -> xyz=1.3500 0.0000 2.2000 rpy=0 0 0
